File: Hardware/continuity.kicad_sch (KiCad schematic)
At the start: 30 parts, among them U6 VN7050ASTR, U7 VN7050ASTR, U8 VN7050ASTR

Commit message: Fáfnir V1.1 redesign
Parts:
- removed D12, D15, D9: LED, LED_SMD:LED_0603_1608Metric_Pad1.05x0.95mm_HandSolder, symbol Device:LED
- removed R29, R34, R39: 100, Resistor_SMD:R_0603_1608Metric, symbol Device:R
Connections:
- net JMPR is gone; now on net +10V: R35.1, U8.5 (VCC), U8.8 (VCC)
- net +10V: now also U7.5 (VCC), U7.8 (VCC)
- net +24V: no longer U7.5 (VCC), U7.8 (VCC)
