File: Hardware/SIGURD.kicad_pcb (KiCad board)
At the start: 4 copper layers, 70 x 70 mm, 116 parts, among them J1 INPUT, J10 24V Terminal, J11 12V/24V Terminal, J12 Extra NF, J2 CAN input, J3 CAN out (optional), J4 jst_sh 4, J5 Step Up Terminal, J6 PWM, J7 Motor Terminal, J8 Hall sensor, J9 12V Terminal, Q1 MMBT3904, U1 TCAN334GDCN, U2 STM32U575CGTx, U3 AMS1117-3.3, U5 LMV324AIDR, U6 VN7050ASTR, U7 VN7050ASTR, U8 VN7050ASTR, U9 AP63205WU, Y1 48MHz

Commit message: Fáfnir V1.1 redesign
Parts:
- removed C14: 0.1u, Capacitor_SMD:C_0603_1608Metric_Pad1.08x0.95mm_HandSolder
- removed C18: 22u, Capacitor_SMD:C_0603_1608Metric_Pad1.08x0.95mm_HandSolder
- removed D8: 3V, Diode_SMD:D_SOD-323_HandSoldering
- removed F2: 5A, Fuse:Fuse_1206_3216Metric
- removed F3: Fuse, Fuse:Fuse_1206_3216Metric
- removed F4, F5, F6: 2.0 A, Fuse:Fuse_1812_4532Metric
- removed FB1: BLM18KG102SN1D, Inductor_SMD:L_0603_1608Metric_Pad1.05x0.95mm_HandSolder
- removed J10: 24V Terminal, TerminalBlock_Phoenix:TerminalBlock_Phoenix_MKDS-1,5-2-5.08_1x02_P5.08mm_Horizontal
- removed J11: 12V/24V Terminal, TerminalBlock_Phoenix:TerminalBlock_Phoenix_MKDS-1,5-2-5.08_1x02_P5.08mm_Horizontal
- removed J12: Extra NF, Connector_PinHeader_2.54mm:PinHeader_1x05_P2.54mm_Vertical
- removed J6: PWM, Connector_JST:JST_XH_B2B-XH-A_1x02_P2.50mm_Vertical
- removed J7: Motor Terminal, TerminalBlock_Phoenix:TerminalBlock_Phoenix_MKDS-1,5-2-5.08_1x02_P5.08mm_Horizontal
- removed J8: Hall sensor, Connector_Molex:Molex_Micro-Fit_3.0_43045-0612_2x03_P3.00mm_Vertical
- removed J9: 12V Terminal, TerminalBlock_Phoenix:TerminalBlock_Phoenix_MKDS-1,5-2-5.08_1x02_P5.08mm_Horizontal
- removed R25: 47k, Resistor_SMD:R_0603_1608Metric_Pad0.98x0.95mm_HandSolder
- removed R39: 100, Resistor_SMD:R_0603_1608Metric
- removed U5: LMV324AIDR, LMV324AIDR:D14_TEX
- removed U8: VN7050ASTR, VN7050ASTR:SOIC_050ASTR_STM
- added C22: 10u, Capacitor_SMD:C_0603_1608Metric, F.Cu at (85.5, 85.7)
- added C23: 0.1u, Capacitor_SMD:C_0201_0603Metric, F.Cu at (79.9, 100.0)
- added C24: SS, Capacitor_SMD:C_0201_0603Metric, F.Cu at (79.1, 106.1)
- added C25: C_comp, Capacitor_SMD:C_0201_0603Metric, F.Cu at (82.7, 106.0)
- added C26: C_HF, Capacitor_SMD:C_0201_0603Metric, F.Cu at (81.6, 105.6)
- added C27: 0.1u, Capacitor_SMD:C_0201_0603Metric, F.Cu at (81.0, 100.3)
- added C28: 4.7u, Capacitor_SMD:C_0402_1005Metric, F.Cu at (78.5, 100.6)
- added C29: 10u, Capacitor_SMD:C_0603_1608Metric, F.Cu at (95.4, 82.9)
- added C30: 0.1u, Capacitor_SMD:C_0201_0603Metric, F.Cu at (89.7, 97.5)
- added C31: 10u, Capacitor_SMD:C_0603_1608Metric, F.Cu at (96.9, 82.9)
- added C32: 0.1u, Capacitor_SMD:C_0402_1005Metric, F.Cu at (98.2, 82.9)
- added C33: 0.47u, Capacitor_SMD:C_0402_1005Metric, F.Cu at (104.6, 80.3)
- added C34: 30p, Capacitor_SMD:C_0402_1005Metric, F.Cu at (105.1, 82.3)
- added C35: 0.1u, Capacitor_SMD:C_0402_1005Metric, F.Cu at (98.2, 80.8)
- added C36: 22u, Capacitor_SMD:C_0603_1608Metric, F.Cu at (107.0, 76.5)
- added C37: 22u, Capacitor_SMD:C_0603_1608Metric, F.Cu at (105.4, 76.5)
- added C38: 1u, Capacitor_SMD:C_0402_1005Metric, F.Cu at (88.8, 97.5)
- added C39: 100p, Capacitor_SMD:C_0201_0603Metric, F.Cu at (82.5, 104.1)
- added C40: 0.1u, Capacitor_SMD:C_0201_0603Metric, F.Cu at (82.9, 103.0)
- added C41: 10u, Capacitor_SMD:C_0603_1608Metric, F.Cu at (87.6, 97.5)
- added C42: 22u, Capacitor_SMD:C_0603_1608Metric, F.Cu at (85.5, 84.2)
- added D17: 28V, Diode_SMD:D_0603_1608Metric_Pad1.05x0.95mm_HandSolder, F.Cu at (103.2, 125.4)
- added D18: 3V, Diode_SMD:D_SOD-323_HandSoldering, F.Cu at (90.5, 117.8)
- added D19: 28V, Diode_SMD:D_0603_1608Metric_Pad1.05x0.95mm_HandSolder, F.Cu at (93.2, 119.3)
- added D20: LED, LED_SMD:LED_0603_1608Metric_Pad1.05x0.95mm_HandSolder, F.Cu at (110.5, 79.0)
- added F10: 2.0 A, Fuse:Fuse_1812_4532Metric, F.Cu at (99.5, 123.3)
- added F11: 2.0 A, Fuse:Fuse_1812_4532Metric, F.Cu at (96.9, 117.2)
- added F7: 2.0 A, Fuse:Fuse_1812_4532Metric, F.Cu at (116.5, 117.2)
- added F8: 2.0 A, Fuse:Fuse_1812_4532Metric, F.Cu at (86.0, 121.4)
- added F9: 2.0 A, Fuse:Fuse_1812_4532Metric, F.Cu at (114.6, 123.3)
- added IC3: TPS56A37RPAR, TPS56A37RPAR:RPA0010A-MFG, F.Cu at (101.2, 82.6)
- added J14: CHANNELS, Connector_Wago:Wago_734-170_1x10_P3.50mm_Horizontal, F.Cu at (89.6, 131.7)
- added JP3: SolderJumper_3_Open, Jumper:SolderJumper-3_P2.0mm_Open_TrianglePad1.0x1.5mm_NumberLabels, F.Cu at (82.3, 112.3)
- added JP4: SolderJumper_3_Open, Jumper:SolderJumper-3_P1.3mm_Open_Pad1.0x1.5mm_NumberLabels, F.Cu at (93.2, 85.3)
- added JP5: SolderJumper_2_Open, Jumper:SolderJumper-2_P1.3mm_Open_RoundedPad1.0x1.5mm, F.Cu at (108.3, 82.2)
- added L2: 10u, FAUL0640-100MT:IND-SMD_L7.0-W6.6_FAUL06XX, F.Cu at (84.1, 90.0)
- added L3: 5.6u, FEXL0660A-5R6M:IND-SMD_L6.6-W6.4, F.Cu at (101.0, 76.5)
- added Q3: CSD17577Q3A, Package_SON:VSON-8_3.3x3.3mm_P0.65mm_NexFET, F.Cu at (80.5, 97.1)
- added Q4: CSD18543Q3A, Package_SON:VSON-8_3.3x3.3mm_P0.65mm_NexFET, F.Cu at (84.8, 97.1)
- added R23: ~, Resistor_SMD:R_0201_0603Metric, F.Cu at (110.3, 104.3)
- added R24: ~, Resistor_SMD:R_0201_0603Metric, F.Cu at (109.5, 104.3)
- added R42: ~, Resistor_SMD:R_0201_0603Metric, F.Cu at (106.1, 104.3)
- added R43: 47k, Resistor_SMD:R_0603_1608Metric_Pad0.98x0.95mm_HandSolder, F.Cu at (86.7, 117.7)
- added R44: 47k, Resistor_SMD:R_0603_1608Metric_Pad0.98x0.95mm_HandSolder, F.Cu at (85.1, 117.6)
- added R45: 10k, Resistor_SMD:R_0201_0603Metric, F.Cu at (75.1, 123.0)
- added R46: 15k, Resistor_SMD:R_0201_0603Metric, F.Cu at (75.1, 121.6)
- added R47: 52.3k, Resistor_SMD:R_0402_1005Metric, F.Cu at (101.6, 85.2)
- added R48: 383k, Resistor_SMD:R_0402_1005Metric, F.Cu at (106.1, 82.3)
- added R49: 20k, Resistor_SMD:R_0402_1005Metric, F.Cu at (104.1, 82.3)
- added R50: 100, Resistor_SMD:R_0402_1005Metric, F.Cu at (89.3, 91.8)
- added U4: INA226, Package_SO:VSSOP-10_3x3mm_P0.5mm, F.Cu at (123.7, 82.8)
- C1: value 4u7 -> 4.7u; footprint Capacitor_SMD:C_0603_1608Metric_Pad1.08x0.95mm_HandSolder -> Capacitor_SMD:C_0201_0603Metric
- C10, C11, C19, C9: footprint Capacitor_SMD:C_0603_1608Metric_Pad1.08x0.95mm_HandSolder -> Capacitor_SMD:C_0201_0603Metric
- C12: value 1u -> 470p; footprint Capacitor_SMD:C_0603_1608Metric_Pad1.08x0.95mm_HandSolder -> Capacitor_SMD:C_0201_0603Metric
- C13: footprint Capacitor_SMD:C_0603_1608Metric_Pad1.08x0.95mm_HandSolder -> Capacitor_SMD:C_0603_1608Metric
- C15: value 1u -> 0.1u; footprint Capacitor_SMD:C_0603_1608Metric_Pad1.08x0.95mm_HandSolder -> Capacitor_SMD:C_0402_1005Metric
- C16, C21: footprint Capacitor_SMD:C_0603_1608Metric_Pad1.08x0.95mm_HandSolder -> Capacitor_SMD:C_0402_1005Metric
- C17: value 10u -> 0.1u; footprint Capacitor_SMD:C_0603_1608Metric_Pad1.08x0.95mm_HandSolder -> Capacitor_SMD:C_0201_0603Metric
- C2: value 4u7 -> 4.7u; footprint Capacitor_SMD:C_0603_1608Metric_Pad1.08x0.95mm_HandSolder -> Capacitor_SMD:C_0402_1005Metric
- C20: value 0.1u -> 1u; footprint Capacitor_SMD:C_0603_1608Metric_Pad1.08x0.95mm_HandSolder -> Capacitor_SMD:C_0402_1005Metric
- C3, C5, C6, C7: value 100n -> 0.1u; footprint Capacitor_SMD:C_0603_1608Metric_Pad1.08x0.95mm_HandSolder -> Capacitor_SMD:C_0201_0603Metric
- C4: value 100n -> 0.1u; footprint Capacitor_SMD:C_0603_1608Metric_Pad1.08x0.95mm_HandSolder -> Capacitor_SMD:C_0402_1005Metric
- D1: footprint Diode_SMD:D_0603_1608Metric_Pad1.05x0.95mm_HandSolder -> Diode_SMD:D_SOD-123
- D10, D16: value 28V -> 3V; footprint Diode_SMD:D_0603_1608Metric_Pad1.05x0.95mm_HandSolder -> Diode_SMD:D_SOD-323_HandSoldering
- D12, D15: value LED -> 28V; footprint LED_SMD:LED_0603_1608Metric_Pad1.05x0.95mm_HandSolder -> Diode_SMD:D_0603_1608Metric_Pad1.05x0.95mm_HandSolder
- J1: footprint Connector_JST:JST_VH_B2P-VH-FB-B_1x02_P3.96mm_Vertical -> Connector_AMASS:AMASS_XT30PW-F_1x02_P2.50mm_Horizontal
- J2, J3: footprint Connector_JST:JST_XH_B2B-XH-AM_1x02_P2.50mm_Vertical -> Connector_JST:JST_XH_B2B-XH-A_1x02_P2.50mm_Vertical
- J5: value Step Up Terminal -> SERVO; footprint TerminalBlock_Phoenix:TerminalBlock_Phoenix_MKDS-1,5-3_1x03_P5.00mm_Horizontal -> Connector_Phoenix_MC:PhoenixContact_MC_1,5_3-GF-3.5_1x03_P3.50mm_Horizontal_ThreadedFlange
- JP2: value Solder jumper -> SolderJumper_3_Open; footprint Jumper:SolderJumper-3_P2.0mm_Open_TrianglePad1.0x1.5mm -> Jumper:SolderJumper-3_P2.0mm_Open_TrianglePad1.0x1.5mm_NumberLabels
- R11, R7, R8, R9: footprint Resistor_SMD:R_0603_1608Metric_Pad0.98x0.95mm_HandSolder -> Resistor_SMD:R_0402_1005Metric
- R16: value 10k -> ~; footprint Resistor_SMD:R_0603_1608Metric_Pad0.98x0.95mm_HandSolder -> Resistor_SMD:R_0201_0603Metric
- R17: value 10k -> RT; footprint Resistor_SMD:R_0603_1608Metric_Pad0.98x0.95mm_HandSolder -> Resistor_SMD:R_0201_0603Metric
- R18: value 10k -> R_comp; footprint Resistor_SMD:R_0603_1608Metric_Pad0.98x0.95mm_HandSolder -> Resistor_SMD:R_0201_0603Metric
- R19: value 15k -> 21k; footprint Resistor_SMD:R_0603_1608Metric_Pad0.98x0.95mm_HandSolder -> Resistor_SMD:R_0201_0603Metric
- R20: value 15k -> 14k; footprint Resistor_SMD:R_0603_1608Metric_Pad0.98x0.95mm_HandSolder -> Resistor_SMD:R_0201_0603Metric
- R21: value 15k -> 0.05; footprint Resistor_SMD:R_0603_1608Metric_Pad0.98x0.95mm_HandSolder -> Resistor_SMD:R_0402_1005Metric
- R26: value 15k -> 1k
- R27, R35: value 47k -> ~; footprint Resistor_SMD:R_0603_1608Metric_Pad0.98x0.95mm_HandSolder -> Resistor_SMD:R_0201_0603Metric
- R28: value 1k -> ~; footprint Resistor_SMD:R_0603_1608Metric_Pad0.98x0.95mm_HandSolder -> Resistor_SMD:R_0201_0603Metric
- R29, R34: value 100 -> 47k; footprint Resistor_SMD:R_0603_1608Metric -> Resistor_SMD:R_0603_1608Metric_Pad0.98x0.95mm_HandSolder
- R30: value 47k -> 1k
- R31, R36: value 15k -> 47k
- R33, R38: value 1k -> 47k
- R6: value 10k -> 0.02; footprint Resistor_SMD:R_0603_1608Metric_Pad0.98x0.95mm_HandSolder -> Resistor_SMD:R_0805_2012Metric
- U3: value AMS1117-3.3 -> LM51231QRGRRQ1; footprint Package_TO_SOT_SMD:SOT-223-3_TabPin2 -> LM51231-Q1:RGR0020C-MFG
- U6: value VN7050ASTR -> TPS4H160AQPWPRQ1; footprint VN7050ASTR:SOIC_050ASTR_STM -> TPS4H160-Q1:PWP0028C_N
- U9: value AP63205WU -> AP63203WU
- Y1: footprint Crystal:Crystal_SMD_0603-4Pin_6.0x3.5mm_HandSoldering -> Crystal:Crystal_SMD_2016-4Pin_2.0x1.6mm
- moved C12 58.2 mm to (78.0, 105.7), turned to 180 degrees
- moved Q1 49.3 mm to (115.3, 110.9), turned to -90 degrees
- moved R6 48.0 mm to (123.7, 78.1), turned to 0 degrees
- moved R2 46.4 mm to (115.3, 108.1), turned to 0 degrees
- moved U3 45.8 mm to (79.8, 103.1)
- moved R3 45.0 mm to (115.3, 106.5), turned to 180 degrees
- moved L1 40.4 mm to (94.0, 95.4)
- moved R26 39.4 mm to (89.2, 104.1)
- moved C19 37.4 mm to (96.1, 94.5), turned to 90 degrees
- moved C16 37.3 mm to (94.0, 96.7), turned to 0 degrees
- moved U9 37.1 mm to (94.0, 92.6), turned to -90 degrees
- moved R7 36.7 mm to (120.9, 83.8), turned to 0 degrees
- moved D9 36.0 mm to (87.5, 104.1), turned to -90 degrees
- moved R9 35.5 mm to (129.3, 104.6)
- moved R30 34.6 mm to (112.2, 79.1), turned to 90 degrees
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Connections:
- net V_input renamed VIN
- C12 pad 1: Earth -> Net-(U3-VREF_RANGE)
- C12 pad 2: Net-(C12-Pad2) -> Earth
- C13 pad 2: Net-(U9-EN) -> +12.8V
- C15 pad 2: Net-(U9-EN) -> +12.8V
- C16 pad 1: 5V -> +3V3
- C17 pad 1: 5V -> +3V3
- C20 pad 2: 5V -> +12.8V
- C21 pad 1: 5V -> +3V3
- D1 pad 2: +10V -> +12.8V
- D10 pad 1: Earth -> /SOL1_SENSE
- D10 pad 2: /SOL1_OUT -> Earth
- D11 pad 1: /SOL2_SENSE -> /IGNI_SENSE
- D12 pad 1: Net-(D12-K) -> Earth
- D12 pad 2: /SOL2_SENSE -> /SOL1_OUT
- D13 pad 2: /SOL2_OUT -> /IGNITION_OUT
- D14 pad 1: /SOL3_SENSE -> /SOL2_SENSE
- D15 pad 1: Net-(D15-K) -> Earth
- D15 pad 2: /SOL3_SENSE -> /SOL2_OUT
- D16 pad 1: Earth -> /SOL3_SENSE
- D16 pad 2: /SOL3_OUT -> Earth
- D9 pad 1: Net-(D9-K) -> Earth
- D9 pad 2: /SOL1_SENSE -> Net-(D9-A)
- F1 pad 2: +10V -> +12.8V
- J5 pad 1: Earth -> Net-(J5-Pin_1)
- J5 pad 2: +24V -> /MOTOR_PWM
- J5 pad 3: +10V -> +12V
- JP2 pad 1: +10V -> +12V
- JP2 pad 2: JMPR -> VS
- L1 pad 2: 5V -> +3V3
- R16 pad 1: /pull_3 -> +3V3
- R16 pad 2: /Hall Sensor Buffer/HALL3 -> Net-(U6-ST3_FAULT_N)
- R17 pad 1: /pull_2 -> Net-(U3-RT)
- R17 pad 2: /Hall Sensor Buffer/HALL2 -> Earth
- R18 pad 1: /pull_1 -> Net-(U3-COMP)
- R18 pad 2: /Hall Sensor Buffer/HALL1 -> Net-(C25-Pad1)
- R19 pad 1: /Hall Sensor Buffer/HALL3 -> Net-(U3-VREF_RANGE)
- R19 pad 2: Earth -> Net-(U3-TRK)
- R20 pad 1: /Hall Sensor Buffer/HALL2 -> Net-(U3-TRK)
- R21 pad 1: /Hall Sensor Buffer/HALL1 -> +12.8V
- R21 pad 2: Earth -> Net-(L2-Pad1)
- R26 pad 1: /SOL1 -> +24V
- R26 pad 2: Earth -> Net-(D9-A)
- R27 pad 1: /SOL1_OUT -> /SOL3
- R27 pad 2: /SOL1_SENSE -> Net-(U6-IN3)
- R28 pad 1: Net-(U6-MULTISENSE) -> /SOL4
- R28 pad 2: Earth -> Net-(U6-IN4)
- R29 pad 1: Net-(D9-K) -> /SOL1_OUT
- R29 pad 2: Earth -> /SOL1_SENSE
- R30 pad 1: +24V -> +12V
- R30 pad 2: /SOL2_OUT -> Net-(D20-A)
- R31 pad 1: /SOL2 -> /SOL2_OUT
- R31 pad 2: Earth -> /SOL2_SENSE
- R32 pad 1: /SOL2_OUT -> /SOL3_OUT
- R32 pad 2: /SOL2_SENSE -> /SOL3_SENSE
- R33 pad 1: Net-(U7-MULTISENSE) -> /SOL4_OUT
- R33 pad 2: Earth -> /SOL4_SENSE
- R34 pad 1: Net-(D12-K) -> VS
- R34 pad 2: Earth -> /SOL1_OUT
- R35 pad 1: JMPR -> Net-(U6-ST4_CS_N)
- R35 pad 2: /SOL3_OUT -> Earth
- R36 pad 1: /SOL3 -> VS
- R36 pad 2: Earth -> /SOL2_OUT
- R37 pad 1: /SOL3_OUT -> VS
- R37 pad 2: /SOL3_SENSE -> /SOL3_OUT
- R38 pad 1: Net-(U8-MULTISENSE) -> VS
- R38 pad 2: Earth -> /SOL4_OUT
- R6 pad 1: 5V -> Net-(J5-Pin_1)
- R6 pad 2: /pull_3 -> Earth
- R7 pad 1: 5V -> +3V3
- R7 pad 2: /pull_2 -> /SDA
- R8 pad 1: 5V -> +3V3
- R8 pad 2: /pull_1 -> /SCL
- U2 pad 10: /LED_R -> unconnected-(U2-PA0-Pad10)
- U2 pad 11: /LED_B -> /LED_R
- U2 pad 12: /LED_G -> /LED_B
- U2 pad 13: /HALL1_buff -> /LED_G
- U2 pad 14: /HALL2_buff -> unconnected-(U2-PA4-Pad14)
- U2 pad 15: /HALL3_buff -> unconnected-(U2-PA5-Pad15)
- U2 pad 16: /MOTOR_PWM -> unconnected-(U2-PA6-Pad16)
- U2 pad 17: /PA7 -> unconnected-(U2-PA7-Pad17)
- U2 pad 18: /PB0 -> unconnected-(U2-PB0-Pad18)
- U2 pad 19: /PB1 -> unconnected-(U2-PB1-Pad19)
- U2 pad 20: /PB2 -> /IGNI_SENSE
- U2 pad 21: /PB10 -> /SOL4_SENSE
- U2 pad 25: unconnected-(U2-PB12-Pad25) -> /SOL3_SENSE
- U2 pad 26: /SOL3_SENSE -> unconnected-(U2-PB13-Pad26)
- U2 pad 29: /SOL1 -> /FAULT
- U2 pad 30: /SOL2 -> /SOL4
- U2 pad 32: unconnected-(U2-PA11-Pad32) -> /SOL2
- U2 pad 33: unconnected-(U2-PA12-Pad33) -> /SOL1
- U2 pad 38: unconnected-(U2-PA15-Pad38) -> /BUZZER
- U2 pad 39: unconnected-(U2-PB3-Pad39) -> /LED_TX
- U2 pad 40: unconnected-(U2-PB4-Pad40) -> /LED_RX
- U2 pad 41: /LED_TX -> unconnected-(U2-PB5-Pad41)
- U2 pad 42: /LED_RX -> /SCL
- U2 pad 43: /BUZZER -> /SDA
- U3 pad 1: Earth -> +12.8V
- U3 pad 2: +3V3 -> Net-(U3-CSN)
- U3 pad 3: 5V -> +24V
- U6 pad 1: /SOL1 -> Earth
- U6 pad 2: Earth -> unconnected-(U6-NC-Pad2)
- U6 pad 3: Earth -> Net-(U6-IN1)
- U6 pad 4: Net-(U6-MULTISENSE) -> Net-(U6-IN2)
- U6 pad 5: +10V -> Net-(U6-IN3)
- U6 pad 6: Net-(F4-Pad2) -> Net-(U6-IN4)
- U6 pad 7: Net-(F4-Pad2) -> unconnected-(U6-ST1_SEH_N-Pad7)
- U6 pad 8: +10V -> unconnected-(U6-ST2_SEL_N-Pad8)
- U7 pad 1: /SOL2 -> /IGNI_1
- U7 pad 2: Earth -> Net-(U7-SEN)
- U7 pad 5: +24V -> /Ignition Channel/VS
- U7 pad 8: +24V -> /Ignition Channel/VS
- U9 pad 1: 5V -> +3V3
- U9 pad 2: Net-(U9-EN) -> +12.8V
- U9 pad 3: Net-(U9-EN) -> +12.8V
Routing:
- net Net-(BZ1-+): track 130.4 -> 20.2 mm, vias 5 -> 0
- net Earth: track 179.6 -> 77.4 mm, vias 64 -> 39
- net 5V: track 94.3 -> 0.00 mm, vias 6 -> 0
- net VS: track 0.00 -> 71.7 mm, vias 0 -> 3
- net +3V3: track 90.4 -> 28.0 mm, vias 9 -> 11
- net /BUZZER: track 64.0 -> 12.3 mm, vias 4 -> 2
- net /MOTOR_PWM: track 35.1 -> 0.00 mm, vias 2 -> 0
- net /SOL4_SENSE: track 0.00 -> 30.9 mm, vias 0 -> 2
- net /IGNI_SENSE: track 0.00 -> 30.2 mm
- net JMPR: track 27.7 -> 0.00 mm, vias 2 -> 0
- net /HALL3_buff: track 24.5 -> 0.00 mm
- net /HALL2_buff: track 23.9 -> 0.00 mm
- net /SOL1: track 27.7 -> 3.99 mm, vias 2 -> 0
- net Net-(U9-EN): track 22.6 -> 0.00 mm, vias 2 -> 0
- net /CAN_H: track 35.4 -> 13.5 mm, vias 2 -> 0
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- added copper zone on B.Cu, net (none)
- added copper zone on F.Cu, net (none)
- added copper zone on F.Cu, net +12.8V
- added copper zone on In2.Cu, net +3V3
- added copper zone on In1.Cu, net Earth
- added copper zone on F.Cu, net SW
- removed copper zone on B.Cu, net +10V
- removed copper zone on F.Cu, net +10V
- removed copper zone on In1.Cu, net +10V
- removed copper zone on In2.Cu, net +10V
- removed copper zone on In1.Cu, net +24V
- removed copper zone on F.Cu, net /SOL1_OUT
- removed copper zone on F.Cu, net /SOL2_OUT
- removed copper zone on F.Cu, net /SOL3_OUT
- removed copper zone on B.Cu, net Earth
- removed copper zone on F.Cu, net Net-(F4-Pad2)
- removed copper zone on F.Cu, net Net-(F8-Pad2)
- removed copper zone on F.Cu, net Net-(J7-Pin_1)
- removed copper zone on B.Cu, net VIN
- removed copper zone on In1.Cu, net VIN
- removed copper zone on In2.Cu, net VIN
Other:
- outline, holes or cut-outs redrawn
- board text added: "Alex Soproni"
- board text added: "Charlie Sandvall"
- board text added: "FÁFNIR V2.0"

Commit message: fafnir redesign :)
Parts:
- removed C20: 1u, Capacitor_SMD:C_0402_1005Metric
- removed G***: LOGO, AESIR LOGO:AESIR LOGO
- added C14: 0.1u, Capacitor_SMD:C_0402_1005Metric, F.Cu at (120.9, 80.8)
- added C43: 10u, Capacitor_SMD:C_0805_2012Metric, F.Cu at (97.4, 88.0)
- added C44: 0.1u, Capacitor_SMD:C_0402_1005Metric, F.Cu at (95.9, 88.0)
- added D21: LED, Diode_SMD:D_0603_1608Metric, F.Cu at (96.5, 77.7)
- added J6: Conn_01x04, Connector_PinSocket_1.27mm:PinSocket_1x04_P1.27mm_Vertical, F.Cu at (104.2, 90.3)
- added R25: 10, Resistor_SMD:R_0402_1005Metric, F.Cu at (121.5, 79.3)
- added R39: 3k, Resistor_SMD:R_0603_1608Metric, F.Cu at (96.5, 74.6)
- added R51: 10, Resistor_SMD:R_0402_1005Metric, F.Cu at (120.5, 79.3)
- added R52: 120, Resistor_SMD:R_0402_1005Metric, F.Cu at (98.7, 90.7)
- added TP1: +24V, TestPoint:TestPoint_Pad_D2.0mm, F.Cu at (75.4, 111.2)
- added TP3: +3V3, TestPoint:TestPoint_Pad_D2.0mm, F.Cu at (75.4, 116.0)
- added TP4: GND, TestPoint:TestPoint_Pad_D2.0mm, F.Cu at (76.0, 85.7)
- added TP5: +12V, TestPoint:TestPoint_Pad_D2.0mm, F.Cu at (129.0, 80.8)
- added TP7: SENSE1, TestPoint:TestPoint_Pad_D2.0mm, F.Cu at (137.8, 125.9)
- BZ1: footprint Buzzer_Beeper:MagneticBuzzer_CUI_CMT-8504-100-SMT -> FEXL0660A-5R6M:BUZ-SMD_4P-L7.5-W7.5-P7.59-TL
- C1, C10, C12, C17, C19, C23, C27, C3, C30, C39, C40, C5, C6, C7, C9: footprint Capacitor_SMD:C_0201_0603Metric -> Capacitor_SMD:C_0402_1005Metric
- C11: value 4u7 -> 4.7u; footprint Capacitor_SMD:C_0201_0603Metric -> Capacitor_SMD:C_0402_1005Metric
- C16, C21, C38: footprint Capacitor_SMD:C_0402_1005Metric -> Capacitor_SMD:C_0603_1608Metric
- C24: value SS -> 330n; footprint Capacitor_SMD:C_0201_0603Metric -> Capacitor_SMD:C_0402_1005Metric
- C25: value C_comp -> 6.8n; footprint Capacitor_SMD:C_0201_0603Metric -> Capacitor_SMD:C_0402_1005Metric
- C26: value C_HF -> 47p; footprint Capacitor_SMD:C_0201_0603Metric -> Capacitor_SMD:C_0402_1005Metric
- C29, C31, C36, C37: footprint Capacitor_SMD:C_0603_1608Metric -> Capacitor_SMD:C_0805_2012Metric
- C42: value 22u -> 10u
- C8: footprint Capacitor_SMD:C_0603_1608Metric_Pad1.08x0.95mm_HandSolder -> Capacitor_SMD:C_0402_1005Metric
- D1: value 28V -> ~
- D10, D11, D14, D16, D18: footprint Diode_SMD:D_SOD-323_HandSoldering -> Diode_SMD:D_SOD-323
- D12, D13, D15, D17, D19: value 28V -> ~; footprint Diode_SMD:D_0603_1608Metric_Pad1.05x0.95mm_HandSolder -> Diode_SMD:D_0603_1608Metric
- D20, D3, D4, D7, D9: footprint LED_SMD:LED_0603_1608Metric_Pad1.05x0.95mm_HandSolder -> Diode_SMD:D_0603_1608Metric
- F10, F11, F7, F8, F9: value 2.0 A -> 1.0A
- J14: footprint Connector_Wago:Wago_734-170_1x10_P3.50mm_Horizontal -> 1935242:CONN10_1935242_PXC
- J4: value jst_sh 4 -> SWD
- J5: footprint Connector_Phoenix_MC:PhoenixContact_MC_1,5_3-GF-3.5_1x03_P3.50mm_Horizontal_ThreadedFlange -> 1727023:CONN_1727023_PXC
- JP5: footprint Jumper:SolderJumper-2_P1.3mm_Open_RoundedPad1.0x1.5mm -> Jumper:SolderJumper-2_P1.3mm_Open_Pad1.0x1.5mm
- L1: value 4.7uH -> 3.9u; footprint Inductor_SMD:L_0603_1608Metric_Pad1.05x0.95mm_HandSolder -> Inductor_SMD:L_Changjiang_FNR4030S
- R1: value 56 -> 100; footprint LED_SMD:LED_0603_1608Metric -> Resistor_SMD:R_0402_1005Metric
- R12, R13, R14, R15, R22, R29, R31, R32, R33, R34, R36, R37, R38, R43, R44: footprint Resistor_SMD:R_0603_1608Metric_Pad0.98x0.95mm_HandSolder -> Resistor_SMD:R_0603_1608Metric
- R16, R35: value ~ -> 10k; footprint Resistor_SMD:R_0201_0603Metric -> Resistor_SMD:R_0402_1005Metric
- R17: value RT -> 49.9k; footprint Resistor_SMD:R_0201_0603Metric -> Capacitor_SMD:C_0402_1005Metric
- R18: value R_comp -> 54.9k; footprint Resistor_SMD:R_0201_0603Metric -> Resistor_SMD:R_0402_1005Metric
- R19: value 21k -> 15k; footprint Resistor_SMD:R_0201_0603Metric -> Resistor_SMD:R_0402_1005Metric
- R20: value 14k -> 10k; footprint Resistor_SMD:R_0201_0603Metric -> Resistor_SMD:R_0402_1005Metric
- R21: value 0.05 -> 0.02; footprint Resistor_SMD:R_0402_1005Metric -> Resistor_SMD:R_2512_6332Metric
- R23, R24, R27, R28, R42: value ~ -> 1k; footprint Resistor_SMD:R_0201_0603Metric -> Resistor_SMD:R_0402_1005Metric
- R26: value 1k -> 7.5k; footprint Resistor_SMD:R_0603_1608Metric_Pad0.98x0.95mm_HandSolder -> Resistor_SMD:R_0603_1608Metric
- R30: value 1k -> 3k; footprint Resistor_SMD:R_0603_1608Metric_Pad0.98x0.95mm_HandSolder -> Resistor_SMD:R_0603_1608Metric
- R4, R5: value ~ -> 1k; footprint Resistor_SMD:R_0603_1608Metric_Pad0.98x0.95mm_HandSolder -> Resistor_SMD:R_0603_1608Metric
- R40: value 22 -> 100; footprint Resistor_SMD:R_0603_1608Metric -> Resistor_SMD:R_0402_1005Metric
- R41: footprint Resistor_SMD:R_0603_1608Metric -> Resistor_SMD:R_0402_1005Metric
- R45, R46: footprint Resistor_SMD:R_0201_0603Metric -> Resistor_SMD:R_0402_1005Metric
- R6: footprint Resistor_SMD:R_0805_2012Metric -> Resistor_SMD:R_2512_6332Metric
- R7, R8: value 10k -> 3.3k
- Y1: value 48MHz -> 24MHz
- moved R22 21.0 mm to (78.6, 116.6), turned to 0 degrees
- moved D7 18.8 mm to (78.6, 115.0), turned to 0 degrees
- moved R50 13.0 mm to (85.3, 104.1), turned to 90 degrees
- moved R26 12.4 mm to (78.5, 110.4), turned to 0 degrees
- moved D9 11.9 mm to (78.5, 112.0), turned to 0 degrees
- moved R8 7.95 mm to (122.5, 90.6)
- moved J14 7.58 mm to (82.2, 133.3)
- moved R7 7.29 mm to (116.7, 89.8), turned to -90 degrees
- moved R6 7.05 mm to (118.0, 82.2), turned to 90 degrees
- moved JP3 5.94 mm to (87.5, 109.4), turned to 90 degrees
- moved D20 5.51 mm to (114.1, 83.2)
- moved JP5 4.78 mm to (106.7, 77.7)
- moved C16 4.35 mm to (94.7, 101.0), turned to -90 degrees
- moved C41 3.70 mm to (91.3, 97.4)
- moved R1 3.50 mm to (102.5, 93.2)
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Connections:
- net Net-(JP5-A) renamed +12VR
- C13 pad 2: +12.8V -> VCC
- C15 pad 2: +12.8V -> VCC
- C22 pad 2: +12.8V -> VCC
- C23 pad 2: +12.8V -> VCC
- C28 pad 2: VCC -> VCC_P
- C39 pad 1: +12.8V -> VCC
- C42 pad 2: +12.8V -> VCC
- D1 pad 2: +12.8V -> VCC
- F1 pad 2: +12.8V -> VCC
- J5 pad 1: Net-(J5-Pin_1) -> /MOTOR_PWM
- J5 pad 2: /MOTOR_PWM -> Net-(J5-Pin_2)
- JP2 pad 1: +12V -> VCC
- JP3 pad 1: +12V -> VCC
- JP4 pad 2: +12.8V -> VCC
- R21 pad 1: +12.8V -> VCC
- R6 pad 1: Net-(J5-Pin_1) -> Earth
- R6 pad 2: Earth -> Net-(J5-Pin_2)
- U2 pad 10: unconnected-(U2-PA0-Pad10) -> /EXT_TX
- U2 pad 11: /LED_R -> /EXT_RX
- U2 pad 12: /LED_B -> unconnected-(U2-PA2-Pad12)
- U2 pad 13: /LED_G -> unconnected-(U2-PA3-Pad13)
- U2 pad 14: unconnected-(U2-PA4-Pad14) -> /LED_R
- U2 pad 15: unconnected-(U2-PA5-Pad15) -> /LED_B
- U2 pad 16: unconnected-(U2-PA6-Pad16) -> /LED_G
- U2 pad 18: unconnected-(U2-PB0-Pad18) -> /MOTOR_PWM
- U2 pad 19: unconnected-(U2-PB1-Pad19) -> /IGNI_SENSE
- U2 pad 20: /IGNI_SENSE -> /SOL4_SENSE
- U2 pad 21: /SOL4_SENSE -> unconnected-(U2-PB10-Pad21)
- U2 pad 26: unconnected-(U2-PB13-Pad26) -> /SOL2_SENSE
- U2 pad 27: /SOL2_SENSE -> /FAULT
- U2 pad 29: /FAULT -> unconnected-(U2-PA8-Pad29)
- U3 pad 1: +12.8V -> VCC
- U3 pad 12: VCC -> VCC_P
- U3 pad 13: +12.8V -> VCC
- U3 pad 22: (no net) -> Earth
- U3 pad 23: (no net) -> Earth
- U3 pad 24: (no net) -> Earth
- U3 pad 25: (no net) -> Earth
- U3 pad 26: (no net) -> Earth
- U3 pad 8: +12.8V -> VCC
- U3 pad 9: VCC -> VCC_P
- U4 pad 10: Net-(J5-Pin_1) -> Net-(U4-Vin+)
- U4 pad 8: 12V -> +12V
- U4 pad 9: Earth -> Net-(U4-Vin-)
- U6 pad 7: unconnected-(U6-ST1_SEH_N-Pad7) -> Earth
- U6 pad 8: unconnected-(U6-ST2_SEL_N-Pad8) -> Earth
- U6 pad V: (no net) -> Earth
- U9 pad 2: +12.8V -> VCC
- U9 pad 3: +12.8V -> VCC
Routing:
- net VCC: track 0.00 -> 154.9 mm, vias 0 -> 15
- net Earth: track 77.4 -> 218.3 mm, vias 39 -> 63
- net +24V: track 5.20 -> 67.0 mm, vias 6 -> 10
- net +12V: track 0.00 -> 43.0 mm, vias 0 -> 1
- net /MOTOR_PWM: track 0.00 -> 33.2 mm, vias 0 -> 1
- net /CAN_H: track 13.5 -> 42.5 mm
- net /SOL1_SENSE: track 25.8 -> 53.6 mm
- net /CAN_L: track 18.0 -> 43.0 mm
- net SW: track 7.21 -> 28.3 mm
- net +3V3: track 28.0 -> 48.8 mm, vias 11 -> 17
- net Net-(L2-Pad1): track 3.48 -> 22.3 mm, vias 0 -> 2
- net /SDA: track 0.00 -> 18.3 mm, vias 0 -> 2
- net /SCL: track 0.00 -> 17.0 mm, vias 0 -> 2
- net /IGNITION_OUT: track 5.96 -> 19.8 mm
- net +12VR: track 7.01 -> 20.8 mm
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- added copper zone on F.Cu, net +12V
- added copper zone on F.Cu, net +12VR
- added copper zone on B.Cu, net +24V
- added copper zone on F.Cu, net Net-(IC3-SW)
- added copper zone on F.Cu, net Net-(IC3-VIN_1)
- added copper zone on F.Cu, net Net-(J5-Pin_2)
- added copper zone on F.Cu, net Net-(L2-Pad1)
- added copper zone on F.Cu, net VCC
- removed copper zone on F.Cu, net +12.8V
Other:
- outline, holes or cut-outs redrawn
- board text added: "+12V"
- board text added: "+24V"
- board text added: "+3V3"
- board text added: "BUCK REG"
- board text added: "CAN"
- board text added: "FÁFNIR"
- board text added: "GND"
- board text added: "H"
- board text added: "IGN"
- board text added: "L"
- board text added: "Robin Sachsenweger Ballantyne"
- board text added: "S1"
- board text added: "S1 SENSE"
- board text added: "S2"
- board text added: "S3"
- board text added: "S4"
- board text added: "SWD"
- board text added: "UART"
- board text added: "V1.1"
- board text removed: "FÁFNIR V2.0"
