File: Hardware/SIGURD.kicad_sch (KiCad schematic)
At the start: 83 parts, among them J1 INPUT, J10 24V Terminal, J11 12V/24V Terminal, J12 Extra NF, J2 CAN input, J3 CAN out (optional), J4 jst_sh 4, J5 Step Up Terminal, J6 PWM, J7 Motor Terminal, J8 Hall sensor, J9 12V Terminal, Q1 MMBT3904, U1 TCAN334GDCN, U2 STM32U575CGTx, U3 AMS1117-3.3, U9 AP63205WU, Y1 48MHz

Commit message: Fáfnir V1.1 redesign
Parts:
- removed C14: 0.1u, Capacitor_SMD:C_0603_1608Metric_Pad1.08x0.95mm_HandSolder, symbol Device:C_Small
- removed C18: 22u, Capacitor_SMD:C_0603_1608Metric_Pad1.08x0.95mm_HandSolder, symbol Device:C_Small
- removed F2: 5A, Fuse:Fuse_1206_3216Metric, symbol Device:Fuse
- removed F3: Fuse, Fuse:Fuse_1206_3216Metric, symbol Device:Fuse
- removed FB1: BLM18KG102SN1D, Inductor_SMD:L_0603_1608Metric_Pad1.05x0.95mm_HandSolder, symbol Device:FerriteBead_Small
- removed J10: 24V Terminal, TerminalBlock_Phoenix:TerminalBlock_Phoenix_MKDS-1,5-2-5.08_1x02_P5.08mm_Horizontal, symbol Connector:Screw_Terminal_01x02
- removed J11: 12V/24V Terminal, TerminalBlock_Phoenix:TerminalBlock_Phoenix_MKDS-1,5-2-5.08_1x02_P5.08mm_Horizontal, symbol Connector:Screw_Terminal_01x02
- removed J12: Extra NF, Connector_PinHeader_2.54mm:PinHeader_1x05_P2.54mm_Vertical, symbol Connector:Conn_01x05_Pin
- removed J5: Step Up Terminal, TerminalBlock_Phoenix:TerminalBlock_Phoenix_MKDS-1,5-3_1x03_P5.00mm_Horizontal, symbol Connector:Screw_Terminal_01x03
- removed J6: PWM, Connector_JST:JST_XH_B2B-XH-A_1x02_P2.50mm_Vertical, symbol Connector_Generic:Conn_01x02
- removed J7: Motor Terminal, TerminalBlock_Phoenix:TerminalBlock_Phoenix_MKDS-1,5-2-5.08_1x02_P5.08mm_Horizontal, symbol Connector:Screw_Terminal_01x02
- removed J8: Hall sensor, Connector_Molex:Molex_Micro-Fit_3.0_43045-0612_2x03_P3.00mm_Vertical, symbol Connector_Generic:Conn_01x06
- removed J9: 12V Terminal, TerminalBlock_Phoenix:TerminalBlock_Phoenix_MKDS-1,5-2-5.08_1x02_P5.08mm_Horizontal, symbol Connector:Screw_Terminal_01x02
- removed R16, R17, R18, R6, R7, R8: 10k, Resistor_SMD:R_0603_1608Metric_Pad0.98x0.95mm_HandSolder, symbol Device:R
- removed R19, R20, R21: 25k, Resistor_SMD:R_0603_1608Metric_Pad0.98x0.95mm_HandSolder, symbol Device:R
- removed U3: AMS1117-3.3, Package_TO_SOT_SMD:SOT-223-3_TabPin2, symbol Regulator_Linear:AMS1117-3.3
- added C20, C38: 1u, Capacitor_SMD:C_0402_1005Metric, symbol Device:C_Small
- added C22, C41: 10u, Capacitor_SMD:C_0603_1608Metric, symbol Device:C_Small
- added C23, C27, C30, C40: 0.1u, Capacitor_SMD:C_0201_0603Metric, symbol Device:C_Small
- added C24: SS, Capacitor_SMD:C_0201_0603Metric, symbol Device:C_Small
- added C25: C_comp, Capacitor_SMD:C_0201_0603Metric, symbol Device:C_Small
- added C26: C_HF, Capacitor_SMD:C_0201_0603Metric, symbol Device:C_Small
- added C28: 4.7u, Capacitor_SMD:C_0402_1005Metric, symbol Device:C_Small
- added C29, C31: 10u, Capacitor_SMD:C_0603_1608Metric, symbol Device:C
- added C32: 0.1u, Capacitor_SMD:C_0402_1005Metric, symbol Device:C
- added C33: 0.47u, Capacitor_SMD:C_0402_1005Metric, symbol Device:C
- added C34: 30p, Capacitor_SMD:C_0402_1005Metric, symbol Device:C
- added C35: 0.1u, Capacitor_SMD:C_0402_1005Metric, symbol Device:C_Small
- added C36, C37: 22u, Capacitor_SMD:C_0603_1608Metric, symbol Device:C
- added C39: 100p, Capacitor_SMD:C_0201_0603Metric, symbol Device:C_Small
- added C42: 22u, Capacitor_SMD:C_0603_1608Metric, symbol Device:C_Small
- added D20, D9: LED, LED_SMD:LED_0603_1608Metric_Pad1.05x0.95mm_HandSolder, symbol Device:LED
- added IC3: TPS56A37RPAR, TPS56A37RPAR:RPA0010A-MFG, symbol SamacSys_Parts:TPS56A37RPAR
- added J14: CHANNELS, Connector_Wago:Wago_734-170_1x10_P3.50mm_Horizontal, symbol Connector_Generic:Conn_01x10
- added J5: SERVO, Connector_Phoenix_MC:PhoenixContact_MC_1,5_3-GF-3.5_1x03_P3.50mm_Horizontal_ThreadedFlange, symbol Connector_Generic:Conn_01x03
- added JP3: SolderJumper_3_Open, Jumper:SolderJumper-3_P2.0mm_Open_TrianglePad1.0x1.5mm_NumberLabels, symbol Jumper:SolderJumper_3_Open
- added JP4: SolderJumper_3_Open, Jumper:SolderJumper-3_P1.3mm_Open_Pad1.0x1.5mm_NumberLabels, symbol Jumper:SolderJumper_3_Open
- added JP5: SolderJumper_2_Open, Jumper:SolderJumper-2_P1.3mm_Open_RoundedPad1.0x1.5mm, symbol Jumper:SolderJumper_2_Open
- added L2: 10u, FAUL0640-100MT:IND-SMD_L7.0-W6.6_FAUL06XX, symbol Device:L_Small
- added L3: 5.6u, FEXL0660A-5R6M:IND-SMD_L6.6-W6.4, symbol Device:L_Small
- added Q3: CSD17577Q3A, Package_SON:VSON-8_3.3x3.3mm_P0.65mm_NexFET, symbol Transistor_FET:CSD17577Q3A
- added Q4: CSD18543Q3A, Package_SON:VSON-8_3.3x3.3mm_P0.65mm_NexFET, symbol Transistor_FET:CSD18543Q3A
- added R16, R23, R24, R27, R28, R35, R42: ~, Resistor_SMD:R_0201_0603Metric, symbol Device:R_Small
- added R17: RT, Resistor_SMD:R_0201_0603Metric, symbol Device:R_Small
- added R18: R_comp, Resistor_SMD:R_0201_0603Metric, symbol Device:R_Small
- added R19: 21k, Resistor_SMD:R_0201_0603Metric, symbol Device:R_Small
- added R20: 14k, Resistor_SMD:R_0201_0603Metric, symbol Device:R_Small
- added R21: 0.05, Resistor_SMD:R_0402_1005Metric, symbol Device:R_Small
- added R26, R30: 1k, Resistor_SMD:R_0603_1608Metric_Pad0.98x0.95mm_HandSolder, symbol Device:R_Small
- added R47: 52.3k, Resistor_SMD:R_0402_1005Metric, symbol Device:R
- added R48: 383k, Resistor_SMD:R_0402_1005Metric, symbol Device:R
- added R49: 20k, Resistor_SMD:R_0402_1005Metric, symbol Device:R
- added R50: 100, Resistor_SMD:R_0402_1005Metric, symbol Device:R_Small
- added R6: 0.02, Resistor_SMD:R_0805_2012Metric, symbol Device:R_Small
- added R7, R8: 10k, Resistor_SMD:R_0402_1005Metric, symbol Device:R_Small
- added U3: LM51231QRGRRQ1, LM51231-Q1:RGR0020C-MFG, symbol LM51231-Q1:LM51231QRGRRQ1
- added U4: INA226, Package_SO:VSSOP-10_3x3mm_P0.5mm, symbol Sensor_Energy:INA226
- added U6: TPS4H160AQPWPRQ1, PWP0028C_N, symbol TPS4H160-Q1:TPS4H160AQPWPRQ1
- C1: value 4u7 -> 4.7u; footprint Capacitor_SMD:C_0603_1608Metric_Pad1.08x0.95mm_HandSolder -> Capacitor_SMD:C_0201_0603Metric
- C10, C11, C19, C9: footprint Capacitor_SMD:C_0603_1608Metric_Pad1.08x0.95mm_HandSolder -> Capacitor_SMD:C_0201_0603Metric
- C12: value 1u -> 470p; footprint Capacitor_SMD:C_0603_1608Metric_Pad1.08x0.95mm_HandSolder -> Capacitor_SMD:C_0201_0603Metric
- C13: footprint Capacitor_SMD:C_0603_1608Metric_Pad1.08x0.95mm_HandSolder -> Capacitor_SMD:C_0603_1608Metric
- C15: value 1u -> 0.1u; footprint Capacitor_SMD:C_0603_1608Metric_Pad1.08x0.95mm_HandSolder -> Capacitor_SMD:C_0402_1005Metric
- C16, C21: footprint Capacitor_SMD:C_0603_1608Metric_Pad1.08x0.95mm_HandSolder -> Capacitor_SMD:C_0402_1005Metric
- C17: value 10u -> 0.1u; footprint Capacitor_SMD:C_0603_1608Metric_Pad1.08x0.95mm_HandSolder -> Capacitor_SMD:C_0201_0603Metric
- C2: value 4u7 -> 4.7u; footprint Capacitor_SMD:C_0603_1608Metric_Pad1.08x0.95mm_HandSolder -> Capacitor_SMD:C_0402_1005Metric
- C3, C5, C6, C7: value 100n -> 0.1u; footprint Capacitor_SMD:C_0603_1608Metric_Pad1.08x0.95mm_HandSolder -> Capacitor_SMD:C_0201_0603Metric
- C4: value 100n -> 0.1u; footprint Capacitor_SMD:C_0603_1608Metric_Pad1.08x0.95mm_HandSolder -> Capacitor_SMD:C_0402_1005Metric
- D1: footprint Diode_SMD:D_0603_1608Metric_Pad1.05x0.95mm_HandSolder -> Diode_SMD:D_SOD-123
- J1: footprint Connector_JST:JST_VH_B2P-VH-FB-B_1x02_P3.96mm_Vertical -> Connector_AMASS:AMASS_XT30PW-F_1x02_P2.50mm_Horizontal
- J2, J3: footprint Connector_JST:JST_XH_B2B-XH-AM_1x02_P2.50mm_Vertical -> Connector_JST:JST_XH_B2B-XH-A_1x02_P2.50mm_Vertical
- JP2: value Solder jumper -> SolderJumper_3_Open; footprint Jumper:SolderJumper-3_P2.0mm_Open_TrianglePad1.0x1.5mm -> Jumper:SolderJumper-3_P2.0mm_Open_TrianglePad1.0x1.5mm_NumberLabels
- R11, R9: footprint Resistor_SMD:R_0603_1608Metric_Pad0.98x0.95mm_HandSolder -> Resistor_SMD:R_0402_1005Metric
- U9: value AP63205WU -> AP63203WU
- Y1: footprint Crystal:Crystal_SMD_0603-4Pin_6.0x3.5mm_HandSoldering -> Crystal:Crystal_SMD_2016-4Pin_2.0x1.6mm
Connections:
- net 5V is gone; now on net +3V3: C16.1, C17.1, C21.1, L1.2, U9.1 (FB)
- net HALL1_buff is gone; now on net LED_G: U2.13 (PA3)
- net +24V: now also C30.1, C38.1, C40.2, C41.1, JP3.3 (B), Q4.5 (D), R26.1, U3.3 (VOUT_SENSE)
- net +3V3: now also R16.1, R7.1, R8.1, U4.6 (VS)
- net BUZZER: now also U2.38 (PA15); no longer U2.43 (PB7)
- net Earth: now also C12.2, C20.1, C22.1, C23.1, C24.2, C25.2, C26.2, C28.1, C29.1, C30.2, C31.1, C32.1, C33.1, C36.1, C37.1, C38.2, C40.1, C41.2, C42.1, D20.1 (K), D9.1 (K), IC3.3 (AGND), IC3.9 (PGND), J14.10 (Pin_10), J14.2 (Pin_2), J14.4 (Pin_4), J14.6 (Pin_6), J14.8 (Pin_8), Q3.1 (S), Q3.2 (S), Q3.3 (S), R17.2, R20.2, R35.2, R47.2, R49.2, R6.2, U3.10 (PGND), U3.14 (SYNC_DITHER_VH), U3.19 (AGND), U3.21 (EP), U4.1 (A1), U4.2 (A0), U4.7 (GND), U4.9 (Vin-), U6.1 (GND), U6.11 (CL), U6.12 (GND), U6.13 (THER), U6.29 (PAD); no longer C12.1
- net LED_B: now also U2.12 (PA2); no longer U2.11 (PA1)
- net LED_G: no longer U2.12 (PA2)
- net LED_R: now also U2.11 (PA1); no longer U2.10 (PA0)
- net LED_RX: now also U2.40 (PB4); no longer U2.42 (PB6)
- net LED_TX: now also U2.39 (PB3); no longer U2.41 (PB5)
- net MOTOR_PWM: now also J5.2 (Pin_2); no longer U2.16 (PA6)
- net SOL1: now also U2.33 (PA12), R23.1; no longer U2.29 (PA8)
- net SOL1_OUT: now also J14.9 (Pin_9)
- net SOL2: now also U2.32 (PA11), R24.1; no longer U2.30 (PA9)
- net SOL2_OUT: now also J14.7 (Pin_7)
- net SOL3: now also R27.1
- net SOL3_OUT: now also J14.5 (Pin_5)
- net SOL3_SENSE: now also U2.25 (PB12); no longer U2.26 (PB13)
- net +12.8V: now reaches C13.2, C15.2, U9.2 (EN), U9.3 (IN)
- net +12.8V: now also D1.2 (A2), F1.2, C20.2, C22.2, C23.2, C39.1, C42.2, JP4.2 (C), R21.1, U3.1 (CSP), U3.13 (UVLO_EN), U3.8 (BIAS)
- removed net +10V: D1.2 (A2), F1.2, JP2.1 (A)
- net HALL2_buff: no longer names the net of U2.14 (PA4)
- net HALL3_buff: no longer names the net of U2.15 (PA5)
- net JMPR renamed VS
- net VS: now also U6.20 (VS), U6.21 (VS), U6.22 (VS), U6.23 (VS)
- net PA7: no longer names the net of U2.17 (PA7)
- net PB0: no longer names the net of U2.18 (PB0)
- net PB1: no longer names the net of U2.19 (PB1)
- net PB10 renamed SOL4_SENSE
- net PB2 renamed IGNI_SENSE
- net V_input renamed VIN
- new net: C35.2, IC3.6 (SW), L3.1
- new net: C34.2, C36.2, C37.2, JP5.1 (A), L3.2, R48.1
- new net: L2.1, R21.2, R50.1
- new net: J5.1 (Pin_1), R6.1, U4.10 (Vin+)
- new net: C26.1, R18.1, U3.20 (COMP)
- new net: C25.1, R18.2
- new net: C29.2, C31.2, C32.2, IC3.11 (VIN_2), IC3.12 (VIN_3), IC3.13 (VIN_4), IC3.8 (VIN_1), JP4.3 (B)
- new net: R35.1, U6.10 (ST4_CS_N)
- new net: R23.2, U6.3 (IN1)
- new net: R24.2, U6.4 (IN2)
- new net: R27.2, U6.5 (IN3)
- new net: R28.2, U6.6 (IN4)
- new net: R16.2, R42.1, U6.9 (ST3_FAULT_N)
- new net: D20.2 (A), R30.2
- new net: C39.2, R50.2, U3.2 (CSN)
- new net: R17.1, U3.15 (RT)
- new net: C12.1, R19.1, U3.16 (VREF_RANGE)
- new net: D9.2 (A), R26.2
- new net: C35.1, IC3.7 (BOOT)
- new net: C27.1, U3.7 (HB)
- new net: R19.2, R20.1, U3.18 (TRK)
- new net: C24.1, U3.17 (SS)
- new net +12V: J5.3 (Pin_3), JP2.1 (A), JP3.1 (A), JP4.1 (A), JP5.2 (B), R30.1
- new net 12V: U4.8 (Vbus)
- new net FAULT: R42.2, U2.29 (PA8)
- new net FB: C34.1, IC3.2 (FB), R48.2, R49.1
- new net HO: Q4.4 (G), U3.5 (HO)
- new net IGNITION_OUT: J14.1 (Pin_1)
- new net Ignition Channel/VS: JP3.2 (C)
- new net LO: Q3.4 (G), U3.11 (LO)
- new net MODE: IC3.10 (MODE), R47.1
- new net SCL: R8.2, U2.42 (PB6), U4.5 (SCL)
- new net SDA: R7.2, U2.43 (PB7), U4.4 (SDA)
- new net SOL4: R28.1, U2.30 (PA9)
- new net SOL4_OUT: J14.3 (Pin_3)
- new net SS: C33.2, IC3.5 (SS)
- new net SW: C27.2, L2.2, Q3.5 (D), Q4.1 (S), Q4.2 (S), Q4.3 (S), U3.6 (SW)
- new net Solenoid Channel 1/T_IN: U6.27 (OUT1), U6.28 (OUT1)
- new net Solenoid Channel 2/T_IN: U6.25 (OUT2), U6.26 (OUT2)
- new net Solenoid Channel 3/T_IN: U6.17 (OUT3), U6.18 (OUT3)
- new net Solenoid Channel 4/T_IN: U6.15 (OUT4), U6.16 (OUT4)
- new net VCC: C28.2, U3.12 (MODE), U3.9 (VCC)
- no-connect marks 10 -> 23
Other:
- removed sheet Continuity Checker
- removed sheet Hall Sensor Buffer
- added sheet Ignition Channel (Ignition.kicad_sch)
- added sheet Solenoid Channel 1 (untitled.kicad_sch)
- added sheet Solenoid Channel 2 (untitled.kicad_sch)
- added sheet Solenoid Channel 3 (untitled.kicad_sch)
- added sheet Solenoid Channel 4 (untitled.kicad_sch)
- note added: "Power +12.8V"
- note added: "SERVO MOTOR"
- note added: "SOLENOID CHANNELS & IGNITION"
- note added: "cloister black font is TUFF"
- note added: "even the edgecuts, align"
- note added: "https://webench.ti.com/power-designer/switching-regulator/select LM51231-Q1"
- note added: "ignition channel"
- note added: "max current: 2A"
- note added: "write silkscreen on the back side + Fáfnir logo"
- note removed: "Hall Pull up resistor"
- note removed: "MOTOR"
- note removed: "Olof said possibly another solenoid?"
- note removed: "SOLENOID SENSOR"
- note removed: "SOLENOIDS"
- note removed: "STEP UP"
- note removed: "Will the current be too high? Current limit on fuses?"
- note removed: "check that the pins are correct"
- note removed: "max current: 1A"
- note removed: "motor max current is 3.65A"
- note removed: "naming"
- moved on the sheet: BZ1, C1, C10, C11, C13, C15, C16, C19, C2, C21, C3, C4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

Commit message: fafnir redesign :)
Parts:
- removed C20: 1u, Capacitor_SMD:C_0402_1005Metric, symbol Device:C_Small
- removed R6: 0.02, Resistor_SMD:R_0805_2012Metric, symbol Device:R_Small
- added C14: 0.1u, Capacitor_SMD:C_0402_1005Metric, symbol Device:C_Small
- added C43: 10u, Capacitor_SMD:C_0805_2012Metric, symbol Device:C
- added C44: 0.1u, Capacitor_SMD:C_0402_1005Metric, symbol Device:C
- added D21: LED, Diode_SMD:D_0603_1608Metric, symbol Device:LED
- added J6: Conn_01x04, Connector_PinSocket_1.27mm:PinSocket_1x04_P1.27mm_Vertical, symbol Connector_Generic:Conn_01x04
- added R25, R51: 10, Resistor_SMD:R_0402_1005Metric, symbol Device:R_Small
- added R39: 3k, Resistor_SMD:R_0603_1608Metric, symbol Device:R_Small
- added R52: 120, Resistor_SMD:R_0402_1005Metric, symbol Device:R_Small
- added R6: 0.02, Resistor_SMD:R_2512_6332Metric, symbol Device:R
- added TP1: +24V, TestPoint:TestPoint_Pad_D2.0mm, symbol Connector:TestPoint
- added TP3: +3V3, TestPoint:TestPoint_Pad_D2.0mm, symbol Connector:TestPoint
- added TP4: GND, TestPoint:TestPoint_Pad_D2.0mm, symbol Connector:TestPoint
- added TP5: +12V, TestPoint:TestPoint_Pad_D2.0mm, symbol Connector:TestPoint
- added TP7: SENSE1, TestPoint:TestPoint_Pad_D2.0mm, symbol Connector:TestPoint
- BZ1: footprint Buzzer_Beeper:MagneticBuzzer_CUI_CMT-8504-100-SMT -> FEXL0660A-5R6M:BUZ-SMD_4P-L7.5-W7.5-P7.59-TL
- C1, C10, C12, C17, C19, C23, C27, C3, C30, C39, C40, C5, C6, C7, C9: footprint Capacitor_SMD:C_0201_0603Metric -> Capacitor_SMD:C_0402_1005Metric
- C11: value 4u7 -> 4.7u; footprint Capacitor_SMD:C_0201_0603Metric -> Capacitor_SMD:C_0402_1005Metric
- C16, C21, C38: footprint Capacitor_SMD:C_0402_1005Metric -> Capacitor_SMD:C_0603_1608Metric
- C24: value SS -> 330n; footprint Capacitor_SMD:C_0201_0603Metric -> Capacitor_SMD:C_0402_1005Metric
- C25: value C_comp -> 6.8n; footprint Capacitor_SMD:C_0201_0603Metric -> Capacitor_SMD:C_0402_1005Metric
- C26: value C_HF -> 47p; footprint Capacitor_SMD:C_0201_0603Metric -> Capacitor_SMD:C_0402_1005Metric
- C29, C31, C36, C37: footprint Capacitor_SMD:C_0603_1608Metric -> Capacitor_SMD:C_0805_2012Metric
- C42: value 22u -> 10u
- C8: footprint Capacitor_SMD:C_0603_1608Metric_Pad1.08x0.95mm_HandSolder -> Capacitor_SMD:C_0402_1005Metric
- D1: value 28V -> ~
- D20, D3, D4, D7, D9: footprint LED_SMD:LED_0603_1608Metric_Pad1.05x0.95mm_HandSolder -> Diode_SMD:D_0603_1608Metric
- J14: footprint Connector_Wago:Wago_734-170_1x10_P3.50mm_Horizontal -> 1935242:CONN10_1935242_PXC
- J4: value jst_sh 4 -> SWD
- J5: footprint Connector_Phoenix_MC:PhoenixContact_MC_1,5_3-GF-3.5_1x03_P3.50mm_Horizontal_ThreadedFlange -> 1727023:CONN_1727023_PXC
- JP5: footprint Jumper:SolderJumper-2_P1.3mm_Open_RoundedPad1.0x1.5mm -> Jumper:SolderJumper-2_P1.3mm_Open_Pad1.0x1.5mm
- L1: value 4.7uH -> 3.9u; footprint Inductor_SMD:L_0603_1608Metric_Pad1.05x0.95mm_HandSolder -> Inductor_SMD:L_Changjiang_FNR4030S
- R1: value 56 -> 100; footprint LED_SMD:LED_0603_1608Metric -> Resistor_SMD:R_0402_1005Metric
- R12, R13, R14, R15, R22: footprint Resistor_SMD:R_0603_1608Metric_Pad0.98x0.95mm_HandSolder -> Resistor_SMD:R_0603_1608Metric
- R16, R35: value ~ -> 10k; footprint Resistor_SMD:R_0201_0603Metric -> Resistor_SMD:R_0402_1005Metric
- R17: value RT -> 49.9k; footprint Resistor_SMD:R_0201_0603Metric -> Capacitor_SMD:C_0402_1005Metric
- R18: value R_comp -> 54.9k; footprint Resistor_SMD:R_0201_0603Metric -> Resistor_SMD:R_0402_1005Metric
- R19: value 21k -> 15k; footprint Resistor_SMD:R_0201_0603Metric -> Resistor_SMD:R_0402_1005Metric
- R20: value 14k -> 10k; footprint Resistor_SMD:R_0201_0603Metric -> Resistor_SMD:R_0402_1005Metric
- R21: value 0.05 -> 0.02; footprint Resistor_SMD:R_0402_1005Metric -> Resistor_SMD:R_2512_6332Metric
- R23, R24, R27, R28, R42: value ~ -> 1k; footprint Resistor_SMD:R_0201_0603Metric -> Resistor_SMD:R_0402_1005Metric
- R26: value 1k -> 7.5k; footprint Resistor_SMD:R_0603_1608Metric_Pad0.98x0.95mm_HandSolder -> Resistor_SMD:R_0603_1608Metric
- R30: value 1k -> 3k; footprint Resistor_SMD:R_0603_1608Metric_Pad0.98x0.95mm_HandSolder -> Resistor_SMD:R_0603_1608Metric
- R4, R5: value ~ -> 1k; footprint Resistor_SMD:R_0603_1608Metric_Pad0.98x0.95mm_HandSolder -> Resistor_SMD:R_0603_1608Metric
- R40: value 22 -> 100; footprint Resistor_SMD:R_0603_1608Metric -> Resistor_SMD:R_0402_1005Metric
- R41: footprint Resistor_SMD:R_0603_1608Metric -> Resistor_SMD:R_0402_1005Metric
- R7, R8: value 10k -> 3.3k
- Y1: value 48MHz -> 24MHz
Connections:
- net +12.8V is gone; now on net VCC: C13.2, C15.2, C22.2, C23.2, C39.1, C42.2, D1.2 (A2), F1.2, JP4.2 (C), R21.1, U3.1 (CSP), U3.13 (UVLO_EN), U3.8 (BIAS), U9.2 (EN), U9.3 (IN)
- net 12V is gone; now on net +12V: U4.8 (Vbus)
- net +12V: now also C43.1, C44.2, TP5.1; no longer JP2.1 (A), JP3.1 (A)
- net +24V: now also TP1.1
- net +3V3: now also R52.2, TP3.1
- net Earth: now also U6.7 (ST1_SEH_N), U6.8 (ST2_SEL_N), C43.2, C44.1, D21.1 (K), J6.3 (Pin_3), R25.2, R6.1, TP4.1; no longer U4.9 (Vin-)
- net FAULT: now also U2.27 (PB14); no longer U2.29 (PA8)
- net IGNI_SENSE: now also U2.19 (PB1); no longer U2.20 (PB2)
- net LED_B: now also U2.15 (PA5); no longer U2.12 (PA2)
- net LED_G: now also U2.16 (PA6); no longer U2.13 (PA3)
- net LED_R: now also U2.14 (PA4); no longer U2.11 (PA1)
- net MOTOR_PWM: now also J5.1 (Pin_1), U2.18 (PB0); no longer J5.2 (Pin_2)
- net SOL1_SENSE: now also TP7.1
- net SOL2_SENSE: now also U2.26 (PB13); no longer U2.27 (PB14)
- net SOL4_SENSE: now also U2.20 (PB2); no longer U2.21 (PB10)
- net VCC: now also JP2.1 (A), JP3.1 (A); no longer C28.2, U3.12 (MODE), U3.9 (VCC)
- net +12VR: now reaches C34.2, C36.2, C37.2, JP5.1 (A), L3.2, R48.1
- net +12VR: now also R39.1
- net at U4.10 (Vin+): now also C14.2, R51.1; no longer J5.1 (Pin_1)
- net EXT_TX: now reaches U2.10 (PA0)
- net EXT_TX: now also J6.1 (Pin_1)
- new net: J6.4 (Pin_4), R52.1
- new net: J5.2 (Pin_2), R51.2, R6.2
- new net: C14.1, R25.1, U4.9 (Vin-)
- new net: D21.2 (A), R39.2
- new net EXT_RX: J6.2 (Pin_2), U2.11 (PA1)
- new net VCC_P: C28.2, U3.12 (MODE), U3.9 (VCC)
- no-connect marks 23 -> 18
Other:
- note added: "Fáfnir logo + alex, charlie, robin"
- note added: "Huaneng MLT-7525"
- note added: "TOGNJING XTM20024000JT00351001"
- note added: "TUOZHAN P4-1615RGYTCA1-0.6T-C"
- note added: "VCC to 12V (with bypass if VCC<12.8V)"
- note added: "Yohey YHR1206SE1WR0002F5"
- note added: "cjiang FNR4030S3R9MT"
- note added: "implement UVLO, and some mosfet switch. maybe comparator"
- note added: "order 1206 fuse from mouser/digi"
- note removed: "Power +12.8V"
- note removed: "cloister black font is TUFF"
- note removed: "even the edgecuts, align"
- note removed: "https://webench.ti.com/power-designer/switching-regulator/select LM51231-Q1"
- note removed: "ignition channel"
- note removed: "write silkscreen on the back side + Fáfnir logo"
- moved on the sheet: D20, J4, JP5, R30
