File: Hardware/untitled.kicad_sch (KiCad schematic)
At the start: 5 parts

Commit message: fafnir redesign :)
Parts:
- D16: footprint Diode_SMD:D_SOD-323_HandSoldering -> Diode_SMD:D_SOD-323
- D17: value 28V -> ~; footprint Diode_SMD:D_0603_1608Metric_Pad1.05x0.95mm_HandSolder -> Diode_SMD:D_0603_1608Metric
- F10: value 2.0 A -> 1.0A
- R32, R37: footprint Resistor_SMD:R_0603_1608Metric_Pad0.98x0.95mm_HandSolder -> Resistor_SMD:R_0603_1608Metric
Other:
- note added: "EATON 0603ESDA-MLP7"
- note added: "LUTE 1812L010/100GR"
- note added: "R+O BZT52C3V3S"
Changed lines of the file:
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@@
 	(generator_version "9.0")
 	(paper "A4")
+	(text "R+O BZT52C3V3S"
+		(exclude_from_sim no)
+		(at 108.458 80.772 0)
+		(effects
+			(font
+				(size 1.27 1.27)
+			)
+		)
+	)
+	(text "LUTE 1812L010/100GR"
+		(exclude_from_sim no)
+		(at 155.702 67.31 0)
+		(effects
+			(font
+				(size 1.27 1.27)
+			)
+		)
+	)
+	(text "EATON 0603ESDA-MLP7"
+		(exclude_from_sim no)
+		(at 137.414 83.566 0)
+		(effects
+			(font
+				(size 1.27 1.27)
+			)
+		)
+	)
 	(junction
 		(at 135.89 69.85)
@@
 			)
 		)
-		(property "Footprint" "Resistor_SMD:R_0603_1608Metric_Pad0.98x0.95mm_HandSolder"
+		(property "Footprint" "Resistor_SMD:R_0603_1608Metric"
 			(at 118.11 69.85 0)
 			(effects
@@
 			)
 		)
-		(property "Value" "2.0 A"
+		(property "Value" "1.0A"
 			(at 142.24 66.04 90)
 			(effects
@@
 			)
 		)
-		(property "Value" "28V"
+		(property "Value" "~"
 			(at 138.43 76.1999 90)
 			(effects
@@
 				)
 				(justify right)
-			)
-		)
-		(property "Footprint" "Diode_SMD:D_0603_1608Metric_Pad1.05x0.95mm_HandSolder"
+				(hide yes)
+			)
+		)
+		(property "Footprint" "Diode_SMD:D_0603_1608Metric"
 			(at 135.89 74.93 0)
 			(effects
@@
 			)
 		)
-		(property "Footprint" "Diode_SMD:D_SOD-323_HandSoldering"
+		(property "Footprint" "Diode_SMD:D_SOD-323"
 			(at 111.76 72.39 90)
 			(effects
@@
 			)
 		)
-		(property "Footprint" "Resistor_SMD:R_0603_1608Metric_Pad0.98x0.95mm_HandSolder"
+		(property "Footprint" "Resistor_SMD:R_0603_1608Metric"
 			(at 125.73 62.23 0)
 			(effects
